File: generated kicad/keyboard.kicad_pcb (KiCad board)
At the start: 2 copper layers, 350.9 x 122.3 mm, 190 parts

Commit message: blackpill footprint added
Parts:
- added REF**: blackpill, my library:blackpill, F.Cu at (452.1, 55.9)
- moved D_11 19.2 mm to (324.0, 43.7)
- moved D_12 19.2 mm to (343.0, 43.7)
- moved D_13 19.2 mm to (362.1, 43.7)
- moved D_16 19.2 mm to (419.2, 43.7)
- moved D_20 19.2 mm to (152.5, 62.7)
- moved D_23 19.2 mm to (209.7, 62.7)
- moved D_25 19.2 mm to (247.8, 62.7)
- moved D_26 19.2 mm to (266.8, 62.7)
- moved D_29 19.2 mm to (324.0, 62.7)
- moved D_30 19.2 mm to (362.1, 62.7)
- moved D_33 19.2 mm to (419.2, 62.7)
- moved D_37 19.2 mm to (162.1, 81.8)
- moved D_39 19.2 mm to (200.2, 81.8)
- moved D_43 19.2 mm to (276.4, 81.8)
- moved D_44 19.2 mm to (295.4, 81.8)
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Routing:
- added copper zone on B.Cu, net (none)
- added copper zone on F.Cu, net (none)

Commit message: wiring done, controller not placed
Parts:
- removed REF**: blackpill, my library:blackpill
- added J1: Conn_02x20_Top_Bottom, my library:blackpill, F.Cu at (466.5, 77.9)
- moved D_68 0.78 mm to (138.1, 120.7)
- moved D_70 0.78 mm to (176.2, 120.7)
- moved D_72 0.78 mm to (214.3, 120.7)
- moved D_73 0.78 mm to (233.4, 120.7)
- moved D_75 0.78 mm to (271.5, 120.7)
- moved D_76 0.78 mm to (290.5, 120.7)
- moved D_78 0.78 mm to (362.0, 120.7)
- moved D_80 0.78 mm to (400.1, 120.7)
- moved D_81 0.78 mm to (419.1, 120.7)
- moved D_67 0.78 mm to (119.1, 120.7)
- moved D_69 0.78 mm to (157.2, 120.7)
- moved D_71 0.78 mm to (195.3, 120.7)
- moved D_74 0.78 mm to (252.4, 120.7)
- moved D_10 0.78 mm to (304.8, 44.5)
- moved D_11 0.78 mm to (323.9, 44.5)
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Connections:
- K_67 pad 1: col1 -> col0
Routing:
- net row1: track 0.00 -> 323.9 mm
- net row0: track 0.00 -> 323.9 mm
- net row2: track 0.00 -> 314.3 mm
- net row5: track 7.44 -> 319.1 mm
- net row3: track 0.00 -> 309.6 mm
- net row4: track 0.00 -> 300.0 mm
- net col13: track 0.00 -> 112.6 mm
- net col3: track 0.00 -> 111.0 mm
- net col4: track 0.00 -> 110.0 mm
- net col11: track 0.00 -> 107.1 mm
- net col0: track 0.00 -> 104.2 mm
- net col14: track 0.00 -> 103.1 mm
- net col12: track 0.00 -> 103.1 mm
- net col1: track 0.00 -> 98.2 mm
- net col17: track 0.00 -> 95.2 mm
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- removed copper zone on B.Cu, net (none)
- removed copper zone on F.Cu, net (none)

Commit message: pcb diodes and keys arranged
Parts:
- removed D_0, D_91, D_92, D_93, D_94: D, Diode_SMD:D_SOD-123
- removed K_0, K_87, K_88, K_89, K_90, K_91, K_92, K_93, K_94: KEYSW, MX_Only:MXOnly-1U-Hotswap
- added SW1: RotaryEncoder_Switch, Rotary_Encoder:RotaryEncoder_Alps_EC12E-Switch_Vertical_H20mm, F.Cu at (419.8, 59.4)
- added SW2: RotaryEncoder_Switch, Rotary_Encoder:RotaryEncoder_Alps_EC12E-Switch_Vertical_H20mm, F.Cu at (438.8, 59.4)
- D_1, D_10, D_11, D_12, D_13, D_14, D_15, D_16, D_17, D_18, D_19, D_2, D_20, D_21, D_22, D_23, D_24, D_25, D_26, D_27, D_28, D_29, D_3, D_30, D_31, D_32, D_33, D_34, D_35, D_36, D_37, D_38, D_39, D_4, D_40, D_41, D_42, D_43, D_44, D_45, D_46, D_47, D_48, D_49, D_5, D_50, D_51, D_52, D_53, D_54, D_55, D_56, D_57, D_58, D_59, D_6, D_60, D_61, D_62, D_63, D_64, D_65, D_66, D_67, D_68, D_69, D_7, D_70, D_71, D_72, D_73, D_74, D_75, D_76, D_77, D_78, D_79, D_8, D_80, D_81, D_82, D_83, D_84, D_85, D_86, D_87, D_88, D_89, D_9, D_90: moved to F.Cu
- K_28: footprint MX_Only:MXOnly-1U-Hotswap -> MX_Only:MXOnly-2U-Hotswap
- K_30: footprint MX_Only:MXOnly-2U-Hotswap -> MX_Only:MXOnly-1U-Hotswap
- K_31, K_44: footprint MX_Only:MXOnly-1U-Hotswap -> MX_Only:MXOnly-1.5U-Hotswap
- K_34: footprint MX_Only:MXOnly-1.5U-Hotswap -> MX_Only:MXOnly-1U-Hotswap
- K_47: footprint MX_Only:MXOnly-1.5U-Hotswap -> MX_Only:MXOnly-1.75U-Hotswap
- K_51: footprint MX_Only:MXOnly-1.75U-Hotswap -> MX_Only:MXOnly-1U-Hotswap
- K_59, K_62: footprint MX_Only:MXOnly-1U-Hotswap -> MX_Only:MXOnly-2.25U-Hotswap
- K_63, K_67: footprint MX_Only:MXOnly-2.25U-Hotswap -> MX_Only:MXOnly-1U-Hotswap
- K_73: footprint MX_Only:MXOnly-1U-Hotswap -> MX_Only:MXOnly-2.75U-Hotswap
- K_75, K_76: footprint MX_Only:MXOnly-1U-Hotswap -> MX_Only:MXOnly-1.25U-Hotswap
- K_78: footprint MX_Only:MXOnly-2.75U-Hotswap -> MX_Only:MXOnly-1.25U-Hotswap
- K_79: footprint MX_Only:MXOnly-1U-Hotswap -> MX_Only:MXOnly-6.25U-Hotswap
- K_82, K_83, K_85: footprint MX_Only:MXOnly-1.25U-Hotswap -> MX_Only:MXOnly-1U-Hotswap
- K_86: footprint MX_Only:MXOnly-6.25U-Hotswap -> MX_Only:MXOnly-1U-Hotswap
- moved D_34 349.2 mm to (454.0, 82.5)
- moved D_17 344.5 mm to (439.7, 70.6), turned to 0 degrees
- moved D_18 338.1 mm to (452.4, 70.6), turned to 0 degrees
- moved K_82 300.4 mm to (388.9, 157.2)
- moved K_83 295.6 mm to (408.0, 157.2)
- moved K_84 293.3 mm to (427.0, 157.2)
- moved K_85 290.9 mm to (446.1, 157.2)
- moved K_15 253.1 mm to (141.3, 81.0)
- moved K_16 253.1 mm to (160.3, 81.0)
- moved D_66 249.0 mm to (173.0, 139.7)
- moved K_86 238.6 mm to (465.1, 157.2)
- moved D_79 230.2 mm to (154.0, 158.8)
- moved K_31 229.6 mm to (146.1, 100.0)
- moved D_80 225.5 mm to (177.8, 158.8)
- moved D_81 225.5 mm to (196.8, 158.8)
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Connections:
- D_1 pad 1: row0 -> col17
- D_10 pad 1: row0 -> col17
- D_11 pad 1: row0 -> col17
- D_12 pad 1: row0 -> col17
- D_13 pad 1: row0 -> col17
- D_14 pad 1: row0 -> col17
- D_15 pad 1: row0 -> col17
- D_16 pad 1: row0 -> col17
- D_17 pad 1: row1 -> col17
- D_18 pad 1: row1 -> col17
- D_2 pad 1: row0 -> col17
- D_3 pad 1: row0 -> col17
- D_34 pad 1: row2 -> row1
- D_4 pad 1: row0 -> col17
- D_5 pad 1: row0 -> col17
- D_6 pad 1: row0 -> col17
- D_66 pad 1: row3 -> row4
- D_7 pad 1: row0 -> col17
- D_79 pad 1: row4 -> row5
- D_8 pad 1: row0 -> col17
- D_80 pad 1: row4 -> row5
- D_81 pad 1: row4 -> row5
- D_9 pad 1: row0 -> col17
- K_1 pad 1: col1 -> col0
- K_10 pad 1: col11 -> col9
- K_11 pad 1: col12 -> col10
- K_12 pad 1: col13 -> col11
- K_13 pad 1: col14 -> col12
- K_14 pad 1: col15 -> col14
- K_15 pad 1: col16 -> col0
- K_15 pad 2: Net-(D_15-A) -> Net-(D_19-A)
- K_16 pad 1: col17 -> col1
- K_16 pad 2: Net-(D_16-A) -> Net-(D_20-A)
- K_17 pad 1: col0 -> col2
- K_17 pad 2: Net-(D_17-A) -> Net-(D_21-A)
- K_18 pad 1: col1 -> col3
- K_18 pad 2: Net-(D_18-A) -> Net-(D_22-A)
- K_19 pad 1: col2 -> col4
- K_19 pad 2: Net-(D_19-A) -> Net-(D_23-A)
- K_2 pad 1: col2 -> col1
- K_20 pad 1: col3 -> col5
- K_20 pad 2: Net-(D_20-A) -> Net-(D_24-A)
- K_21 pad 1: col4 -> col6
- K_21 pad 2: Net-(D_21-A) -> Net-(D_25-A)
- K_22 pad 1: col5 -> col7
- K_22 pad 2: Net-(D_22-A) -> Net-(D_26-A)
- K_23 pad 1: col6 -> col8
- K_23 pad 2: Net-(D_23-A) -> Net-(D_27-A)
- K_24 pad 1: col7 -> col9
- K_24 pad 2: Net-(D_24-A) -> Net-(D_28-A)
- K_25 pad 1: col8 -> col10
- K_25 pad 2: Net-(D_25-A) -> Net-(D_29-A)
- K_26 pad 1: col9 -> col11
- K_26 pad 2: Net-(D_26-A) -> Net-(D_30-A)
- K_27 pad 1: col10 -> col12
- K_27 pad 2: Net-(D_27-A) -> Net-(D_31-A)
- K_28 pad 1: col11 -> col14
- K_28 pad 2: Net-(D_28-A) -> Net-(D_32-A)
- K_29 pad 1: col12 -> col17
- K_29 pad 2: Net-(D_29-A) -> Net-(D_33-A)
- K_3 pad 1: col4 -> col2
- K_30 pad 1: col14 -> col20
- K_30 pad 2: Net-(D_30-A) -> Net-(D_34-A)
- K_31 pad 1: col15 -> col0
- K_31 pad 2: Net-(D_31-A) -> Net-(D_35-A)
- K_32 pad 1: col16 -> col2
- K_32 pad 2: Net-(D_32-A) -> Net-(D_36-A)
- K_33 pad 1: col17 -> col3
- K_33 pad 2: Net-(D_33-A) -> Net-(D_37-A)
- K_34 pad 1: col0 -> col4
- K_34 pad 2: Net-(D_34-A) -> Net-(D_38-A)
- K_35 pad 1: col2 -> col5
- K_35 pad 2: Net-(D_35-A) -> Net-(D_39-A)
- K_36 pad 1: col3 -> col6
- K_36 pad 2: Net-(D_36-A) -> Net-(D_40-A)
- K_37 pad 1: col4 -> col7
- K_37 pad 2: Net-(D_37-A) -> Net-(D_41-A)
- K_38 pad 1: col5 -> col8
- K_38 pad 2: Net-(D_38-A) -> Net-(D_42-A)
- K_39 pad 1: col6 -> col9
- K_39 pad 2: Net-(D_39-A) -> Net-(D_43-A)
- K_4 pad 1: col5 -> col3
- K_40 pad 1: col7 -> col10
- K_40 pad 2: Net-(D_40-A) -> Net-(D_44-A)
- K_41 pad 1: col8 -> col11
- K_41 pad 2: Net-(D_41-A) -> Net-(D_45-A)
- K_42 pad 1: col9 -> col12
- K_42 pad 2: Net-(D_42-A) -> Net-(D_46-A)
- K_43 pad 1: col10 -> Net-(K_43-COL)
- K_43 pad 2: Net-(D_43-A) -> Net-(D_47-A)
- K_44 pad 1: col11 -> col14
- K_44 pad 2: Net-(D_44-A) -> Net-(D_48-A)
- K_45 pad 1: col12 -> col17
- K_45 pad 2: Net-(D_45-A) -> Net-(D_49-A)
- K_46 pad 1: col13 -> col20
- K_46 pad 2: Net-(D_46-A) -> Net-(D_50-A)
- K_47 pad 1: col14 -> col0
- K_47 pad 2: Net-(D_47-A) -> Net-(D_51-A)
- K_48 pad 1: col15 -> col2
- K_48 pad 2: Net-(D_48-A) -> Net-(D_52-A)
- K_49 pad 1: col16 -> col3
- K_49 pad 2: Net-(D_49-A) -> Net-(D_53-A)
- K_5 pad 1: col6 -> col4
- K_50 pad 1: col17 -> col4
- K_50 pad 2: Net-(D_50-A) -> Net-(D_54-A)
- K_51 pad 1: col0 -> col5
- K_51 pad 2: Net-(D_51-A) -> Net-(D_55-A)
- K_52 pad 1: col2 -> col6
- K_52 pad 2: Net-(D_52-A) -> Net-(D_56-A)
- K_53 pad 1: col3 -> col7
- K_53 pad 2: Net-(D_53-A) -> Net-(D_57-A)
- K_54 pad 1: col4 -> col8
- K_54 pad 2: Net-(D_54-A) -> Net-(D_58-A)
- K_55 pad 1: col5 -> col9
- K_55 pad 2: Net-(D_55-A) -> Net-(D_59-A)
- K_56 pad 1: col6 -> col10
- K_56 pad 2: Net-(D_56-A) -> Net-(D_60-A)
- K_57 pad 1: col7 -> col11
- K_57 pad 2: Net-(D_57-A) -> Net-(D_61-A)
- K_58 pad 1: col8 -> col12
- K_58 pad 2: Net-(D_58-A) -> Net-(D_62-A)
- K_59 pad 1: col9 -> Net-(K_43-COL)
- K_59 pad 2: Net-(D_59-A) -> Net-(D_63-A)
- K_6 pad 1: col7 -> col5
- K_60 pad 1: col10 -> col17
- K_60 pad 2: Net-(D_60-A) -> Net-(D_64-A)
- K_61 pad 1: col11 -> col20
- K_61 pad 2: Net-(D_61-A) -> Net-(D_65-A)
- K_62 pad 1: col12 -> col0
- K_62 pad 2: Net-(D_62-A) -> Net-(D_66-A)
- K_63 pad 1: col13 -> col2
- K_63 pad 2: Net-(D_63-A) -> Net-(D_67-A)
- K_64 pad 1: col15 -> col3
- K_64 pad 2: Net-(D_64-A) -> Net-(D_68-A)
- K_65 pad 1: col16 -> col4
- K_65 pad 2: Net-(D_65-A) -> Net-(D_69-A)
- K_66 pad 1: col17 -> col5
- K_66 pad 2: Net-(D_66-A) -> Net-(D_70-A)
- K_67 pad 1: col0 -> col6
- K_67 pad 2: Net-(D_67-A) -> Net-(D_71-A)
- K_68 pad 1: col2 -> col7
- K_68 pad 2: Net-(D_68-A) -> Net-(D_72-A)
- K_69 pad 1: col3 -> col8
- K_69 pad 2: Net-(D_69-A) -> Net-(D_73-A)
- K_7 pad 1: col8 -> col6
- K_70 pad 1: col4 -> col9
- K_70 pad 2: Net-(D_70-A) -> Net-(D_74-A)
- K_71 pad 1: col5 -> col10
- K_71 pad 2: Net-(D_71-A) -> Net-(D_75-A)
- K_72 pad 1: col6 -> col11
- K_72 pad 2: Net-(D_72-A) -> Net-(D_76-A)
- K_73 pad 1: col7 -> Net-(K_43-COL)
- K_73 pad 2: Net-(D_73-A) -> Net-(D_77-A)
- K_74 pad 1: col8 -> col20
- K_74 pad 2: Net-(D_74-A) -> Net-(D_78-A)
- K_75 pad 1: col9 -> col0
- K_75 pad 2: Net-(D_75-A) -> Net-(D_79-A)
- K_76 pad 1: col10 -> col1
- K_76 pad 2: Net-(D_76-A) -> Net-(D_80-A)
- K_77 pad 1: col11 -> col3
- K_77 pad 2: Net-(D_77-A) -> Net-(D_81-A)
- K_78 pad 1: col13 -> col4
- K_78 pad 2: Net-(D_78-A) -> Net-(D_82-A)
- K_79 pad 1: col15 -> col7
- K_79 pad 2: Net-(D_79-A) -> Net-(D_83-A)
- K_8 pad 1: col9 -> col7
- K_80 pad 1: col16 -> col11
- K_80 pad 2: Net-(D_80-A) -> Net-(D_84-A)
- K_81 pad 1: col17 -> col12
- K_81 pad 2: Net-(D_81-A) -> Net-(D_85-A)
- K_82 pad 1: col0 -> Net-(K_43-COL)
- K_82 pad 2: Net-(D_82-A) -> Net-(D_86-A)
- K_83 pad 1: col1 -> col14
- K_83 pad 2: Net-(D_83-A) -> Net-(D_87-A)
- K_84 pad 1: col3 -> col17
- K_84 pad 2: Net-(D_84-A) -> Net-(D_88-A)
- K_85 pad 1: col4 -> col20
- K_85 pad 2: Net-(D_85-A) -> Net-(D_89-A)
- K_86 pad 1: col7 -> col21
- K_86 pad 2: Net-(D_86-A) -> Net-(D_90-A)
- K_9 pad 1: col10 -> col8
Routing:
- net row1: track 323.9 -> 0.00 mm
- net row0: track 323.9 -> 0.00 mm
- net row5: track 319.1 -> 0.00 mm
- net row2: track 314.3 -> 0.00 mm
- net row3: track 309.6 -> 0.00 mm
- net row4: track 300.0 -> 0.00 mm
- net col13: track 112.6 -> 0.00 mm
- net col3: track 111.0 -> 0.00 mm
- net col4: track 110.0 -> 0.00 mm
- net col11: track 107.1 -> 0.00 mm
- net col0: track 104.2 -> 0.00 mm
- net col14: track 103.1 -> 0.00 mm
- net col12: track 103.1 -> 0.00 mm
- net col1: track 98.2 -> 0.00 mm
- net col17: track 95.2 -> 0.00 mm
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Other:
- board outline removed

Commit message: swapped diodes to front
Parts:
- D_1, D_10, D_11, D_12, D_13, D_14, D_15, D_16, D_17, D_18, D_19, D_2, D_20, D_21, D_22, D_23, D_24, D_25, D_26, D_27, D_28, D_29, D_3, D_30, D_31, D_32, D_33, D_34, D_35, D_36, D_37, D_38, D_39, D_4, D_40, D_41, D_42, D_43, D_44, D_45, D_46, D_47, D_48, D_49, D_5, D_50, D_51, D_52, D_53, D_54, D_55, D_56, D_57, D_58, D_59, D_6, D_60, D_61, D_62, D_63, D_64, D_65, D_66, D_67, D_68, D_69, D_7, D_70, D_71, D_72, D_73, D_74, D_75, D_76, D_77, D_78, D_79, D_8, D_80, D_81, D_82, D_83, D_84, D_85, D_86, D_87, D_88, D_89, D_9, D_90: moved to B.Cu
- turned D_15 to 180 degrees
- turned D_16 to 180 degrees
- turned D_17 to 180 degrees
- turned D_18 to 180 degrees
Routing:
- net col0: track 0.00 -> 1.27 mm

Commit message: routed tracks and fixed accidental intersection near R1
Parts:
- moved D_18 1.80 mm to (453.2, 69.1), turned to 90 degrees
- moved D_15 1.77 mm to (419.9, 69.1), turned to 90 degrees
- moved D_17 1.77 mm to (438.9, 69.1), turned to 90 degrees
- moved D_16 1.73 mm to (434.2, 69.1), turned to 90 degrees
Connections:
- D_1 pad 1: col17 -> row0
- D_10 pad 1: col17 -> row0
- D_11 pad 1: col17 -> row0
- D_12 pad 1: col17 -> row0
- D_13 pad 1: col17 -> row0
- D_14 pad 1: col17 -> row0
- D_15 pad 1: col17 -> row0
- D_16 pad 1: col17 -> row0
- D_17 pad 1: col17 -> row0
- D_18 pad 1: col17 -> row0
- D_2 pad 1: col17 -> row0
- D_3 pad 1: col17 -> row0
- D_4 pad 1: col17 -> row0
- D_5 pad 1: col17 -> row0
- D_6 pad 1: col17 -> row0
- D_7 pad 1: col17 -> row0
- D_8 pad 1: col17 -> row0
- D_9 pad 1: col17 -> row0
Routing:
- net row5: track 0.00 -> 319.1 mm
- net row0: track 0.00 -> 307.2 mm
- net row1: track 0.00 -> 304.8 mm
- net row2: track 0.00 -> 295.3 mm
- net row3: track 0.00 -> 290.5 mm
- net row4: track 0.00 -> 281.0 mm
- net col3: track 0.00 -> 111.0 mm
- net col4: track 0.00 -> 110.0 mm
- net col12: track 0.00 -> 107.7 mm
- net col11: track 0.00 -> 107.1 mm
- net col7: track 0.00 -> 106.1 mm
- net col0: track 1.27 -> 105.4 mm
- net col14: track 0.00 -> 103.1 mm
- net col17: track 0.00 -> 101.1 mm
- net col20: track 0.00 -> 101.1 mm
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
Commit message: stable but not enough pins
Parts:
- added D_91: D, Diode_SMD:D_SOD-123, B.Cu at (457.2, 120.6)
- added D_92: D, Diode_SMD:D_SOD-123, B.Cu at (459.6, 139.8)
- added H2: MountingHole, MountingHole:MountingHole_2.2mm_M2, F.Cu at (478.6, 170.7)
- added H4: MountingHole, MountingHole:MountingHole_2.2mm_M2, F.Cu at (127.8, 170.7)
- added H5: MountingHole, MountingHole:MountingHole_2.2mm_M2, F.Cu at (127.8, 48.4)
- added H6: MountingHole, MountingHole:MountingHole_2.2mm_M2, F.Cu at (478.6, 48.4)
- added SW3: RotaryEncoder_Switch, Rotary_Encoder:RotaryEncoder_Alps_EC12E-Switch_Vertical_H20mm, F.Cu at (468.4, 112.6)
- J1: moved to B.Cu
- moved J1 98.2 mm to (465.9, 78.8)
Connections:
- K_86 pad 1: col21 -> col23
Routing:
- net col23: track 0.00 -> 31.8 mm, vias 0 -> 1
- net row4: track 281.0 -> 303.4 mm
- net Net-(D_92-A): track 0.00 -> 13.6 mm
- net Net-(D_91-A): track 0.00 -> 11.4 mm
- net Net-(D_36-A): track 12.3 -> 5.89 mm
- net col12: track 107.7 -> 103.3 mm, vias 0 -> 8
- net col20: track 101.1 -> 102.9 mm, vias 0 -> 9
- net col17: track 101.1 -> 102.8 mm, vias 0 -> 7
- net col14: track 103.1 -> 103.9 mm, vias 0 -> 6
- net col0: track 105.4 -> 106.1 mm, vias 0 -> 10
- net Net-(K_43-COL): track 68.3 -> 68.6 mm, vias 0 -> 6
- net col7: track 106.1 -> 106.3 mm, vias 0 -> 10
- net col4: track 110.0 -> 110.3 mm, vias 0 -> 10
- net col3: track 111.0 -> 111.3 mm, vias 0 -> 10
- net col11: track 107.1 -> 107.3 mm, vias 0 -> 10
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Other:
- board outline added: 364.5 x 134.3 mm

Commit message: need to flip pcb and fix footprint
Parts:
- added Dc_1: D, Diode_SMD:D_SOD-123, B.Cu at (141.3, 249.3)
- added Dc_10: D, Diode_SMD:D_SOD-123, B.Cu at (312.7, 249.3)
- added Dc_11: D, Diode_SMD:D_SOD-123, B.Cu at (331.8, 249.3)
- added Dc_12: D, Diode_SMD:D_SOD-123, B.Cu at (350.8, 249.3)
- added Dc_13: D, Diode_SMD:D_SOD-123, B.Cu at (369.9, 249.3)
- added Dc_14: D, Diode_SMD:D_SOD-123, B.Cu at (408.0, 249.3)
- added Dc_15: D, Diode_SMD:D_SOD-123, B.Cu at (141.3, 268.4)
- added Dc_16: D, Diode_SMD:D_SOD-123, B.Cu at (160.3, 268.4)
- added Dc_17: D, Diode_SMD:D_SOD-123, B.Cu at (179.4, 268.4)
- added Dc_18: D, Diode_SMD:D_SOD-123, B.Cu at (198.4, 268.4)
- added Dc_19: D, Diode_SMD:D_SOD-123, B.Cu at (217.5, 268.4)
- added Dc_2: D, Diode_SMD:D_SOD-123, B.Cu at (160.3, 249.3)
- added Dc_20: D, Diode_SMD:D_SOD-123, B.Cu at (236.5, 268.4)
- added Dc_21: D, Diode_SMD:D_SOD-123, B.Cu at (255.6, 268.4)
- added Dc_22: D, Diode_SMD:D_SOD-123, B.Cu at (274.6, 268.4)
- added Dc_23: D, Diode_SMD:D_SOD-123, B.Cu at (293.7, 268.4)
- added Dc_24: D, Diode_SMD:D_SOD-123, B.Cu at (312.7, 268.4)
- added Dc_25: D, Diode_SMD:D_SOD-123, B.Cu at (331.8, 268.4)
- added Dc_26: D, Diode_SMD:D_SOD-123, B.Cu at (350.8, 268.4)
- added Dc_27: D, Diode_SMD:D_SOD-123, B.Cu at (369.9, 268.4)
- added Dc_28: D, Diode_SMD:D_SOD-123, B.Cu at (398.5, 268.4)
- added Dc_29: D, Diode_SMD:D_SOD-123, B.Cu at (427.0, 268.3)
- added Dc_3: D, Diode_SMD:D_SOD-123, B.Cu at (179.4, 249.3)
- added Dc_30: D, Diode_SMD:D_SOD-123, B.Cu at (446.1, 268.3)
- added Dc_31: D, Diode_SMD:D_SOD-123, B.Cu at (146.1, 287.4)
- added Dc_32: D, Diode_SMD:D_SOD-123, B.Cu at (169.9, 287.4)
- added Dc_33: D, Diode_SMD:D_SOD-123, B.Cu at (188.9, 287.4)
- added Dc_34: D, Diode_SMD:D_SOD-123, B.Cu at (208.0, 287.4)
- added Dc_35: D, Diode_SMD:D_SOD-123, B.Cu at (227.0, 287.4)
- added Dc_36: D, Diode_SMD:D_SOD-123, B.Cu at (246.1, 287.4)
- added Dc_37: D, Diode_SMD:D_SOD-123, B.Cu at (265.1, 287.4)
- added Dc_38: D, Diode_SMD:D_SOD-123, B.Cu at (284.2, 287.4)
- added Dc_39: D, Diode_SMD:D_SOD-123, B.Cu at (303.2, 287.4)
- added Dc_4: D, Diode_SMD:D_SOD-123, B.Cu at (198.4, 249.3)
- added Dc_40: D, Diode_SMD:D_SOD-123, B.Cu at (322.3, 287.4)
- added Dc_41: D, Diode_SMD:D_SOD-123, B.Cu at (341.3, 287.4)
- added Dc_42: D, Diode_SMD:D_SOD-123, B.Cu at (360.4, 287.4)
- added Dc_43: D, Diode_SMD:D_SOD-123, B.Cu at (379.4, 287.4)
- added Dc_44: D, Diode_SMD:D_SOD-123, B.Cu at (403.2, 287.4)
- added Dc_45: D, Diode_SMD:D_SOD-123, B.Cu at (427.0, 287.4)
- added Dc_46: D, Diode_SMD:D_SOD-123, B.Cu at (446.1, 287.4)
- added Dc_47: D, Diode_SMD:D_SOD-123, B.Cu at (148.4, 306.4)
- added Dc_48: D, Diode_SMD:D_SOD-123, B.Cu at (174.6, 306.4)
- added Dc_49: D, Diode_SMD:D_SOD-123, B.Cu at (193.7, 306.4)
- added Dc_5: D, Diode_SMD:D_SOD-123, B.Cu at (217.5, 249.3)
- added Dc_50: D, Diode_SMD:D_SOD-123, B.Cu at (212.7, 306.4)
- added Dc_51: D, Diode_SMD:D_SOD-123, B.Cu at (231.8, 306.4)
- added Dc_52: D, Diode_SMD:D_SOD-123, B.Cu at (250.8, 306.4)
- added Dc_53: D, Diode_SMD:D_SOD-123, B.Cu at (269.9, 306.4)
- added Dc_54: D, Diode_SMD:D_SOD-123, B.Cu at (288.9, 306.4)
- added Dc_55: D, Diode_SMD:D_SOD-123, B.Cu at (308.0, 306.4)
- added Dc_56: D, Diode_SMD:D_SOD-123, B.Cu at (327.0, 306.4)
- added Dc_57: D, Diode_SMD:D_SOD-123, B.Cu at (346.1, 306.4)
- added Dc_58: D, Diode_SMD:D_SOD-123, B.Cu at (365.1, 306.4)
- added Dc_59: D, Diode_SMD:D_SOD-123, B.Cu at (396.1, 306.5)
- added Dc_6: D, Diode_SMD:D_SOD-123, B.Cu at (236.5, 249.3)
- added Dc_60: D, Diode_SMD:D_SOD-123, B.Cu at (427.0, 306.5)
- added Dc_61: D, Diode_SMD:D_SOD-123, B.Cu at (446.1, 306.5)
- added Dc_62: D, Diode_SMD:D_SOD-123, B.Cu at (153.2, 325.5)
- added Dc_63: D, Diode_SMD:D_SOD-123, B.Cu at (184.2, 325.5)
- added Dc_64: D, Diode_SMD:D_SOD-123, B.Cu at (203.2, 325.5)
- added Dc_65: D, Diode_SMD:D_SOD-123, B.Cu at (222.2, 325.5)
- added Dc_66: D, Diode_SMD:D_SOD-123, B.Cu at (241.3, 325.5)
- added Dc_67: D, Diode_SMD:D_SOD-123, B.Cu at (260.4, 325.5)
- added Dc_68: D, Diode_SMD:D_SOD-123, B.Cu at (279.4, 325.5)
- added Dc_69: D, Diode_SMD:D_SOD-123, B.Cu at (298.4, 325.5)
- added Dc_7: D, Diode_SMD:D_SOD-123, B.Cu at (255.6, 249.3)
- added Dc_70: D, Diode_SMD:D_SOD-123, B.Cu at (317.5, 325.5)
- added Dc_71: D, Diode_SMD:D_SOD-123, B.Cu at (336.6, 325.5)
- added Dc_72: D, Diode_SMD:D_SOD-123, B.Cu at (355.6, 325.5)
- added Dc_73: D, Diode_SMD:D_SOD-123, B.Cu at (391.3, 325.5)
- added Dc_74: D, Diode_SMD:D_SOD-123, B.Cu at (446.1, 325.5)
- added Dc_75: D, Diode_SMD:D_SOD-123, B.Cu at (143.7, 344.6)
- added Dc_76: D, Diode_SMD:D_SOD-123, B.Cu at (167.5, 344.6)
- added Dc_77: D, Diode_SMD:D_SOD-123, B.Cu at (188.9, 344.5)
- added Dc_78: D, Diode_SMD:D_SOD-123, B.Cu at (210.3, 344.6)
- added Dc_79: D, Diode_SMD:D_SOD-123, B.Cu at (281.8, 344.6)
- added Dc_8: D, Diode_SMD:D_SOD-123, B.Cu at (274.6, 249.3)
- added Dc_80: D, Diode_SMD:D_SOD-123, B.Cu at (350.8, 344.6)
- added Dc_81: D, Diode_SMD:D_SOD-123, B.Cu at (369.9, 344.6)
- added Dc_82: D, Diode_SMD:D_SOD-123, B.Cu at (388.9, 344.6)
- added Dc_83: D, Diode_SMD:D_SOD-123, B.Cu at (408.0, 344.6)
- added Dc_84: D, Diode_SMD:D_SOD-123, B.Cu at (427.0, 344.6)
- added Dc_85: D, Diode_SMD:D_SOD-123, B.Cu at (446.1, 344.6)
- added Dc_86: D, Diode_SMD:D_SOD-123, B.Cu at (465.1, 344.6)
- added Dc_87: D, Diode_SMD:D_SOD-123, B.Cu at (412.8, 255.6)
- added Dc_88: D, Diode_SMD:D_SOD-123, B.Cu at (425.4, 255.6)
- added Dc_89: D, Diode_SMD:D_SOD-123, B.Cu at (431.8, 255.6)
- added Dc_9: D, Diode_SMD:D_SOD-123, B.Cu at (293.7, 249.3)
- added Dc_90: D, Diode_SMD:D_SOD-123, B.Cu at (444.5, 255.6)
- added Dc_91: D, Diode_SMD:D_SOD-123, B.Cu at (450.1, 298.4)
- added H1: MountingHole, MountingHole:MountingHole_2.2mm_M2, F.Cu at (342.6, 387.9)
- added H3: MountingHole, MountingHole:MountingHole_2.2mm_M2, F.Cu at (336.7, 387.9)
- added H7: MountingHole, MountingHole:MountingHole_2.2mm_M2, F.Cu at (330.7, 387.9)
- added H8: MountingHole, MountingHole:MountingHole_2.2mm_M2, F.Cu at (324.8, 387.9)
- added J2: Conn_02x20_Top_Bottom, my library:blackpill, F.Cu at (463.6, 264.8)
- added Kc_1: KEYSW, MX_Only:MXOnly-1U-Hotswap, F.Cu at (133.3, 247.7)
- added Kc_10: KEYSW, MX_Only:MXOnly-1U-Hotswap, F.Cu at (304.8, 247.7)
- added Kc_11: KEYSW, MX_Only:MXOnly-1U-Hotswap, F.Cu at (323.9, 247.7)
- added Kc_12: KEYSW, MX_Only:MXOnly-1U-Hotswap, F.Cu at (342.9, 247.7)
- added Kc_13: KEYSW, MX_Only:MXOnly-1U-Hotswap, F.Cu at (361.9, 247.7)
- added Kc_14: KEYSW, MX_Only:MXOnly-1U-Hotswap, F.Cu at (400.1, 247.7)
- added Kc_15: KEYSW, MX_Only:MXOnly-1U-Hotswap, F.Cu at (133.3, 266.7)
- added Kc_16: KEYSW, MX_Only:MXOnly-1U-Hotswap, F.Cu at (152.4, 266.7)
- added Kc_17: KEYSW, MX_Only:MXOnly-1U-Hotswap, F.Cu at (171.4, 266.7)
- added Kc_18: KEYSW, MX_Only:MXOnly-1U-Hotswap, F.Cu at (190.5, 266.7)
- added Kc_19: KEYSW, MX_Only:MXOnly-1U-Hotswap, F.Cu at (209.6, 266.7)
- added Kc_2: KEYSW, MX_Only:MXOnly-1U-Hotswap, F.Cu at (152.4, 247.7)
- added Kc_20: KEYSW, MX_Only:MXOnly-1U-Hotswap, F.Cu at (228.6, 266.7)
- added Kc_21: KEYSW, MX_Only:MXOnly-1U-Hotswap, F.Cu at (247.7, 266.7)
- added Kc_22: KEYSW, MX_Only:MXOnly-1U-Hotswap, F.Cu at (266.7, 266.7)
- added Kc_23: KEYSW, MX_Only:MXOnly-1U-Hotswap, F.Cu at (285.8, 266.7)
- added Kc_24: KEYSW, MX_Only:MXOnly-1U-Hotswap, F.Cu at (304.8, 266.7)
- added Kc_25: KEYSW, MX_Only:MXOnly-1U-Hotswap, F.Cu at (323.9, 266.7)
- added Kc_26: KEYSW, MX_Only:MXOnly-1U-Hotswap, F.Cu at (342.9, 266.7)
- added Kc_27: KEYSW, MX_Only:MXOnly-1U-Hotswap, F.Cu at (361.9, 266.7)
- added Kc_28: KEYSW, MX_Only:MXOnly-2U-Hotswap, F.Cu at (390.5, 266.7)
- added Kc_29: KEYSW, MX_Only:MXOnly-1U-Hotswap, F.Cu at (419.1, 266.7)
- added Kc_3: KEYSW, MX_Only:MXOnly-1U-Hotswap, F.Cu at (171.4, 247.7)
- added Kc_30: KEYSW, MX_Only:MXOnly-1U-Hotswap, F.Cu at (438.1, 266.7)
- added Kc_31: KEYSW, MX_Only:MXOnly-1.5U-Hotswap, F.Cu at (138.1, 285.8)
- added Kc_32: KEYSW, MX_Only:MXOnly-1U-Hotswap, F.Cu at (161.9, 285.8)
- added Kc_33: KEYSW, MX_Only:MXOnly-1U-Hotswap, F.Cu at (181.0, 285.8)
- added Kc_34: KEYSW, MX_Only:MXOnly-1U-Hotswap, F.Cu at (200.0, 285.8)
- added Kc_35: KEYSW, MX_Only:MXOnly-1U-Hotswap, F.Cu at (219.1, 285.8)
- added Kc_36: KEYSW, MX_Only:MXOnly-1U-Hotswap, F.Cu at (238.1, 285.8)
- added Kc_37: KEYSW, MX_Only:MXOnly-1U-Hotswap, F.Cu at (257.2, 285.8)
- added Kc_38: KEYSW, MX_Only:MXOnly-1U-Hotswap, F.Cu at (276.2, 285.8)
- added Kc_39: KEYSW, MX_Only:MXOnly-1U-Hotswap, F.Cu at (295.3, 285.8)
- added Kc_4: KEYSW, MX_Only:MXOnly-1U-Hotswap, F.Cu at (190.5, 247.7)
- added Kc_40: KEYSW, MX_Only:MXOnly-1U-Hotswap, F.Cu at (314.3, 285.8)
- added Kc_41: KEYSW, MX_Only:MXOnly-1U-Hotswap, F.Cu at (333.4, 285.8)
- added Kc_42: KEYSW, MX_Only:MXOnly-1U-Hotswap, F.Cu at (352.4, 285.8)
- added Kc_43: KEYSW, MX_Only:MXOnly-1U-Hotswap, F.Cu at (371.5, 285.8)
- added Kc_44: KEYSW, MX_Only:MXOnly-1.5U-Hotswap, F.Cu at (395.3, 285.8)
- added Kc_45: KEYSW, MX_Only:MXOnly-1U-Hotswap, F.Cu at (419.1, 285.8)
- added Kc_46: KEYSW, MX_Only:MXOnly-1U-Hotswap, F.Cu at (438.1, 285.8)
- added Kc_47: KEYSW, MX_Only:MXOnly-1.75U-Hotswap, F.Cu at (140.5, 304.8)
- added Kc_48: KEYSW, MX_Only:MXOnly-1U-Hotswap, F.Cu at (166.7, 304.8)
- added Kc_49: KEYSW, MX_Only:MXOnly-1U-Hotswap, F.Cu at (185.7, 304.8)
- added Kc_5: KEYSW, MX_Only:MXOnly-1U-Hotswap, F.Cu at (209.6, 247.7)
- added Kc_50: KEYSW, MX_Only:MXOnly-1U-Hotswap, F.Cu at (204.8, 304.8)
- added Kc_51: KEYSW, MX_Only:MXOnly-1U-Hotswap, F.Cu at (223.8, 304.8)
- added Kc_52: KEYSW, MX_Only:MXOnly-1U-Hotswap, F.Cu at (242.9, 304.8)
- added Kc_53: KEYSW, MX_Only:MXOnly-1U-Hotswap, F.Cu at (261.9, 304.8)
- added Kc_54: KEYSW, MX_Only:MXOnly-1U-Hotswap, F.Cu at (281.0, 304.8)
- added Kc_55: KEYSW, MX_Only:MXOnly-1U-Hotswap, F.Cu at (300.0, 304.8)
- added Kc_56: KEYSW, MX_Only:MXOnly-1U-Hotswap, F.Cu at (319.1, 304.8)
- added Kc_57: KEYSW, MX_Only:MXOnly-1U-Hotswap, F.Cu at (338.1, 304.8)
- added Kc_58: KEYSW, MX_Only:MXOnly-1U-Hotswap, F.Cu at (357.2, 304.8)
- added Kc_59: KEYSW, MX_Only:MXOnly-2.25U-Hotswap, F.Cu at (388.1, 304.8)
- added Kc_6: KEYSW, MX_Only:MXOnly-1U-Hotswap, F.Cu at (228.6, 247.7)
- added Kc_60: KEYSW, MX_Only:MXOnly-1U-Hotswap, F.Cu at (419.1, 304.8)
- added Kc_61: KEYSW, MX_Only:MXOnly-1U-Hotswap, F.Cu at (438.1, 304.8)
- added Kc_62: KEYSW, MX_Only:MXOnly-2.25U-Hotswap, F.Cu at (145.3, 323.9)
- added Kc_63: KEYSW, MX_Only:MXOnly-1U-Hotswap, F.Cu at (176.2, 323.9)
- added Kc_64: KEYSW, MX_Only:MXOnly-1U-Hotswap, F.Cu at (195.3, 323.9)
- added Kc_65: KEYSW, MX_Only:MXOnly-1U-Hotswap, F.Cu at (214.3, 323.9)
- added Kc_66: KEYSW, MX_Only:MXOnly-1U-Hotswap, F.Cu at (233.4, 323.9)
- added Kc_67: KEYSW, MX_Only:MXOnly-1U-Hotswap, F.Cu at (252.4, 323.9)
- added Kc_68: KEYSW, MX_Only:MXOnly-1U-Hotswap, F.Cu at (271.5, 323.9)
- added Kc_69: KEYSW, MX_Only:MXOnly-1U-Hotswap, F.Cu at (290.5, 323.9)
- added Kc_7: KEYSW, MX_Only:MXOnly-1U-Hotswap, F.Cu at (247.7, 247.7)
- added Kc_70: KEYSW, MX_Only:MXOnly-1U-Hotswap, F.Cu at (309.6, 323.9)
- added Kc_71: KEYSW, MX_Only:MXOnly-1U-Hotswap, F.Cu at (328.6, 323.9)
- added Kc_72: KEYSW, MX_Only:MXOnly-1U-Hotswap, F.Cu at (347.7, 323.9)
- added Kc_73: KEYSW, MX_Only:MXOnly-2.75U-Hotswap, F.Cu at (383.4, 323.9)
- added Kc_74: KEYSW, MX_Only:MXOnly-1U-Hotswap, F.Cu at (438.1, 323.9)
- added Kc_75: KEYSW, MX_Only:MXOnly-1.25U-Hotswap, F.Cu at (135.7, 342.9)
- added Kc_76: KEYSW, MX_Only:MXOnly-1.25U-Hotswap, F.Cu at (159.5, 342.9)
- added Kc_77: KEYSW, MX_Only:MXOnly-1U-Hotswap, F.Cu at (181.0, 342.9)
- added Kc_78: KEYSW, MX_Only:MXOnly-1.25U-Hotswap, F.Cu at (202.4, 342.9)
- added Kc_79: KEYSW, MX_Only:MXOnly-6.25U-Hotswap, F.Cu at (273.8, 342.9)
- added Kc_8: KEYSW, MX_Only:MXOnly-1U-Hotswap, F.Cu at (266.7, 247.7)
- added Kc_80: KEYSW, MX_Only:MXOnly-1U-Hotswap, F.Cu at (342.9, 342.9)
- added Kc_81: KEYSW, MX_Only:MXOnly-1U-Hotswap, F.Cu at (361.9, 342.9)
- added Kc_82: KEYSW, MX_Only:MXOnly-1U-Hotswap, F.Cu at (381.0, 342.9)
- added Kc_83: KEYSW, MX_Only:MXOnly-1U-Hotswap, F.Cu at (400.1, 342.9)
- added Kc_84: KEYSW, MX_Only:MXOnly-1U-Hotswap, F.Cu at (419.1, 342.9)
- added Kc_85: KEYSW, MX_Only:MXOnly-1U-Hotswap, F.Cu at (438.1, 342.9)
- added Kc_86: KEYSW, MX_Only:MXOnly-1U-Hotswap, F.Cu at (457.2, 342.9)
- added Kc_9: KEYSW, MX_Only:MXOnly-1U-Hotswap, F.Cu at (285.8, 247.7)
- added SWc1: RotaryEncoder_Switch, Rotary_Encoder:RotaryEncoder_Alps_EC12E-Switch_Vertical_H20mm, F.Cu at (411.9, 244.4)
- added SWc2: RotaryEncoder_Switch, Rotary_Encoder:RotaryEncoder_Alps_EC12E-Switch_Vertical_H20mm, F.Cu at (430.9, 244.4)
- added SWc3: RotaryEncoder_Switch, Rotary_Encoder:RotaryEncoder_Alps_EC12E-Switch_Vertical_H20mm, F.Cu at (462.0, 296.5)
Routing:
- net /12x8/COL1: track 0.00 -> 539.0 mm
- net /12x8/COL2: track 0.00 -> 502.0 mm
- net /12x8/COL3: track 0.00 -> 456.6 mm
- net /12x8/COL4: track 0.00 -> 401.5 mm
- net /12x8/ROW11: track 0.00 -> 381.1 mm, vias 0 -> 9
- net /12x8/ROW5: track 0.00 -> 363.2 mm, vias 0 -> 15
- net /12x8/COL5: track 0.00 -> 352.8 mm
- net /12x8/ROW7: track 0.00 -> 351.1 mm, vias 0 -> 15
- net /12x8/ROW9: track 0.00 -> 348.8 mm, vias 0 -> 13
- net /12x8/ROW3: track 0.00 -> 338.8 mm, vias 0 -> 15
- net /12x8/ROW1: track 0.00 -> 322.4 mm, vias 0 -> 15
- net /12x8/COL6: track 0.00 -> 314.4 mm
- net /12x8/COL7: track 0.00 -> 275.9 mm
- net /12x8/COL8: track 0.00 -> 215.2 mm
- net /12x8/ROW10: track 0.00 -> 205.1 mm, vias 0 -> 12
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Other:
- board size 364.5 x 134.3 mm -> 361.9 x 133.3 mm
