File: generated kicad/keyboard.kicad_pcb (KiCad board)
At the start: 2 copper layers, 361.9 x 133.3 mm, 371 parts, among them J1 Conn_02x20_Top_Bottom, J2 Conn_02x20_Top_Bottom, SW1 RotaryEncoder_Switch, SW2 RotaryEncoder_Switch, SW3 RotaryEncoder_Switch

Commit message: fully done with fab no logo
Parts:
- removed D_1, D_10, D_11, D_12, D_13, D_14, D_15, D_16, D_17, D_18, D_19, D_2, D_20, D_21, D_22, D_23, D_24, D_25, D_26, D_27, D_28, D_29, D_3, D_30, D_31, D_32, D_33, D_34, D_35, D_36, D_37, D_38, D_39, D_4, D_40, D_41, D_42, D_43, D_44, D_45, D_46, D_47, D_48, D_49, D_5, D_50, D_51, D_52, D_53, D_54, D_55, D_56, D_57, D_58, D_59, D_6, D_60, D_61, D_62, D_63, D_64, D_65, D_66, D_67, D_68, D_69, D_7, D_70, D_71, D_72, D_73, D_74, D_75, D_76, D_77, D_78, D_79, D_8, D_80, D_81, D_82, D_83, D_84, D_85, D_86, D_87, D_88, D_89, D_9, D_90, D_91, D_92: D, Diode_SMD:D_SOD-123
- removed J1: Conn_02x20_Top_Bottom, my library:blackpill
- removed K_1, K_10, K_11, K_12, K_13, K_14, K_15, K_16, K_17, K_18, K_19, K_2, K_20, K_21, K_22, K_23, K_24, K_25, K_26, K_27, K_29, K_3, K_30, K_32, K_33, K_34, K_35, K_36, K_37, K_38, K_39, K_4, K_40, K_41, K_42, K_43, K_45, K_46, K_48, K_49, K_5, K_50, K_51, K_52, K_53, K_54, K_55, K_56, K_57, K_58, K_6, K_60, K_61, K_63, K_64, K_65, K_66, K_67, K_68, K_69, K_7, K_70, K_71, K_72, K_74, K_77, K_8, K_80, K_81, K_82, K_83, K_84, K_85, K_86, K_9: KEYSW, MX_Only:MXOnly-1U-Hotswap
- removed K_28: KEYSW, MX_Only:MXOnly-2U-Hotswap
- removed K_31, K_44: KEYSW, MX_Only:MXOnly-1.5U-Hotswap
- removed K_47: KEYSW, MX_Only:MXOnly-1.75U-Hotswap
- removed K_59, K_62: KEYSW, MX_Only:MXOnly-2.25U-Hotswap
- removed K_73: KEYSW, MX_Only:MXOnly-2.75U-Hotswap
- removed K_75, K_76, K_78: KEYSW, MX_Only:MXOnly-1.25U-Hotswap
- removed K_79: KEYSW, MX_Only:MXOnly-6.25U-Hotswap
- removed SW1, SW2, SW3: RotaryEncoder_Switch, Rotary_Encoder:RotaryEncoder_Alps_EC12E-Switch_Vertical_H20mm
- H1, H2, H3, H4, H5, H6, H7, H8: footprint MountingHole:MountingHole_2.2mm_M2 -> MountingHole:MountingHole_4.3mm_M4
- J2: moved to B.Cu
- moved H6 346.2 mm to (296.5, 342.9)
- moved H5 319.4 mm to (251.5, 342.9)
- moved H3 268.2 mm to (118.1, 232.4)
- moved H7 197.5 mm to (208.9, 232.4)
- moved H4 187.7 mm to (118.1, 358.1)
- moved H8 168.9 mm to (390.5, 232.4)
- moved H1 141.9 mm to (481.3, 358.1)
- moved H2 61.8 mm to (481.3, 232.4)
- moved Dc_29 0.06 mm to (427.0, 268.4)
- moved Dc_30 0.06 mm to (446.1, 268.4)
- turned J2 to 180 degrees
Connections:
- J2 pad 1: /12x8/ROW2 -> unconnected-(J2-Pin_1-Pad1)
- J2 pad 10: /12x8/ROW5 -> /12x8/COL2
- J2 pad 11: /12x8/ROW7 -> unconnected-(J2-Pin_11-Pad11)
- J2 pad 12: /12x8/ROW9 -> /12x8/COL3
- J2 pad 13: /12x8/ROW11 -> /12x8/COL4
- J2 pad 14: /12x8/ROW8 -> /12x8/COL5
- J2 pad 15: /12x8/ROW10 -> /12x8/ROT3A
- J2 pad 16: /12x8/ROW12 -> unconnected-(J2-Pin_16-Pad16)
- J2 pad 17: /12x8/ROT3A -> /12x8/COL6
- J2 pad 18: unconnected-(J2-Pin_18-Pad18) -> /12x8/COL7
- J2 pad 19: unconnected-(J2-Pin_19-Pad19) -> /12x8/COL8
- J2 pad 2: /12x8/ROW4 -> unconnected-(J2-Pin_2-Pad2)
- J2 pad 21: unconnected-(J2-Pin_21-Pad21) -> /12x8/ROW2
- J2 pad 22: unconnected-(J2-Pin_22-Pad22) -> /12x8/ROW4
- J2 pad 23: unconnected-(J2-Pin_23-Pad23) -> /12x8/ROW6
- J2 pad 24: /12x8/ROT2B -> /12x8/ROW1
- J2 pad 25: unconnected-(J2-Pin_25-Pad25) -> /12x8/ROW3
- J2 pad 26: /12x8/ROT2A -> unconnected-(J2-Pin_26-Pad26)
- J2 pad 27: /12x8/ROT1B -> unconnected-(J2-Pin_27-Pad27)
- J2 pad 28: /12x8/ROT1A -> unconnected-(J2-Pin_28-Pad28)
- J2 pad 29: /12x8/COL5 -> unconnected-(J2-Pin_29-Pad29)
- J2 pad 3: /12x8/ROW6 -> unconnected-(J2-Pin_3-Pad3)
- J2 pad 30: /12x8/COL6 -> /12x8/ROW5
- J2 pad 31: unconnected-(J2-Pin_31-Pad31) -> /12x8/ROW7
- J2 pad 32: /12x8/COL7 -> /12x8/ROW9
- J2 pad 33: /12x8/COL8 -> /12x8/ROW11
- J2 pad 34: /12x8/COL4 -> /12x8/ROW8
- J2 pad 35: /12x8/ROT3B -> /12x8/ROW10
- J2 pad 36: unconnected-(J2-Pin_36-Pad36) -> /12x8/ROW12
- J2 pad 37: /12x8/COL3 -> /12x8/ROT3B
- J2 pad 38: /12x8/COL2 -> unconnected-(J2-Pin_38-Pad38)
- J2 pad 39: /12x8/COL1 -> unconnected-(J2-Pin_39-Pad39)
- J2 pad 4: /12x8/ROW1 -> /12x8/ROT2B
- J2 pad 5: /12x8/ROW3 -> unconnected-(J2-Pin_5-Pad5)
- J2 pad 6: unconnected-(J2-Pin_6-Pad6) -> /12x8/ROT2A
- J2 pad 7: unconnected-(J2-Pin_7-Pad7) -> /12x8/ROT1B
- J2 pad 8: unconnected-(J2-Pin_8-Pad8) -> /12x8/ROT1A
- J2 pad 9: unconnected-(J2-Pin_9-Pad9) -> /12x8/COL1
- SWc1 pad A: /12x8/ROT1B -> /12x8/ROT1A
- SWc1 pad B: /12x8/ROT1A -> /12x8/ROT1B
- SWc2 pad A: /12x8/ROW2B -> /12x8/ROT2A
- SWc2 pad B: /12x8/ROT2A -> /12x8/ROT2B
- SWc3 pad A: /12x8/ROT3B -> /12x8/ROT3A
- SWc3 pad B: /12x8/ROT3A -> /12x8/ROT3B
Routing:
- net row5: track 319.1 -> 0.00 mm
- net row0: track 307.2 -> 0.00 mm
- net row1: track 304.8 -> 0.00 mm
- net row4: track 303.4 -> 0.00 mm
- net row2: track 295.3 -> 0.00 mm
- net row3: track 290.5 -> 0.00 mm
- net /12x8/COL8: track 215.2 -> 436.4 mm, vias 0 -> 1
- net /12x8/COL7: track 275.9 -> 450.0 mm, vias 0 -> 1
- net /12x8/COL6: track 314.4 -> 472.6 mm, vias 0 -> 1
- net /12x8/COL5: track 352.8 -> 500.5 mm, vias 0 -> 1
- net /12x8/COL4: track 401.5 -> 533.3 mm, vias 0 -> 1
- net /12x8/COL3: track 456.6 -> 572.3 mm, vias 0 -> 1
- net col3: track 111.3 -> 0.00 mm, vias 10 -> 0
- net col4: track 110.3 -> 0.00 mm, vias 10 -> 0
- net col11: track 107.3 -> 0.00 mm, vias 10 -> 0
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- added copper zone on B.Cu, net (none)
- added copper zone on F.Cu, net (none)
Other:
- board size 361.9 x 133.3 mm -> 372.1 x 134.6 mm
- board text added: "14650"
- board text added: "1775"
- board text added: "3575"
- board text added: "4950"
- board text added: "5250"
- board text added: "5300"
- board text added: "600"
- board text added: "7150"
- board text added: "7275"
