File: generated kicad/untitled.kicad_sch (KiCad schematic)
At the start: 185 parts, among them J2 Conn_02x20_Top_Bottom

Commit message: fully done with fab no logo
Parts:
- added H2, H4, H5, H6: MountingHole, MountingHole:MountingHole_4.3mm_M4, symbol Mechanical:MountingHole
- H1, H3, H7, H8: footprint MountingHole:MountingHole_2.2mm_M2 -> MountingHole:MountingHole_4.3mm_M4
Connections:
- net ROW2B is gone; now on net ROT2A: SWc2.A
- net COL1: now also J2.9 (Pin_9); no longer J2.39 (Pin_39)
- net COL2: now also J2.10 (Pin_10); no longer J2.38 (Pin_38)
- net COL3: now also J2.12 (Pin_12); no longer J2.37 (Pin_37)
- net COL4: now also J2.13 (Pin_13); no longer J2.34 (Pin_34)
- net COL5: now also J2.14 (Pin_14); no longer J2.29 (Pin_29)
- net COL6: now also J2.17 (Pin_17); no longer J2.30 (Pin_30)
- net COL7: now also J2.18 (Pin_18); no longer J2.32 (Pin_32)
- net COL8: now also J2.19 (Pin_19); no longer J2.33 (Pin_33)
- net ROT1A: now also J2.8 (Pin_8), SWc1.A; no longer J2.28 (Pin_28), SWc1.B
- net ROT1B: now also J2.7 (Pin_7), SWc1.B; no longer J2.27 (Pin_27), SWc1.A
- net ROT2A: now also J2.6 (Pin_6); no longer J2.26 (Pin_26), SWc2.B
- net ROT2B: now also J2.4 (Pin_4), SWc2.B; no longer J2.24 (Pin_24)
- net ROT3A: now also J2.15 (Pin_15), SWc3.A; no longer J2.17 (Pin_17), SWc3.B
- net ROT3B: now also J2.37 (Pin_37), SWc3.B; no longer J2.35 (Pin_35), SWc3.A
- net ROW1: now also J2.24 (Pin_24); no longer J2.4 (Pin_4)
- net ROW10: now also J2.35 (Pin_35); no longer J2.15 (Pin_15)
- net ROW11: now also J2.33 (Pin_33); no longer J2.13 (Pin_13)
- net ROW12: now also J2.36 (Pin_36); no longer J2.16 (Pin_16)
- net ROW2: now also J2.21 (Pin_21); no longer J2.1 (Pin_1)
- net ROW3: now also J2.25 (Pin_25); no longer J2.5 (Pin_5)
- net ROW4: now also J2.22 (Pin_22); no longer J2.2 (Pin_2)
- net ROW5: now also J2.30 (Pin_30); no longer J2.10 (Pin_10)
- net ROW6: now also J2.23 (Pin_23); no longer J2.3 (Pin_3)
- net ROW7: now also J2.31 (Pin_31); no longer J2.11 (Pin_11)
- net ROW8: now also J2.34 (Pin_34); no longer J2.14 (Pin_14)
- net ROW9: now also J2.32 (Pin_32); no longer J2.12 (Pin_12)
Other:
- moved on the sheet: H1, H3, H7, H8
